File: projects/5v radio/5v radio/5v radio.kicad_pcb (KiCad board)
At the start: 2 copper layers, 8 parts, among them U1 NRF24L01_Breakout, U2 LD1117V33

Commit message: 5v radio done
Parts:
- removed U1: NRF24L01_Breakout, RF_Module:nRF24L01_Breakout
- removed U2: LD1117V33, Package_TO_SOT_THT:TO-220-3_Horizontal_TabDown
- removed U3: ~, Footprints_cez:1.3_0.91 inch Oled screen
- removed U4: ~, Footprints_cez:ps_2 connector
- added 3v3_regulator1: LD1117V33, Package_TO_SOT_THT:TO-220-3_Horizontal_TabDown, F.Cu at (120.7, 41.9)
- added NRF24: NRF24L01_Breakout, Footprints_cez:nRF24L01_big, F.Cu at (131.4, 33.0)
- added Oled_screen1: ~, Footprints_cez:1.3inch Oled screen, F.Cu at (124.8, 98.6)
- added ps/2_connector1: ~, Footprints_cez:ps_2 connector, F.Cu at (159.9, 119.1)
- A1: footprint Module:Arduino_Nano -> Footprints_cez:Arduino nano breakout
- moved C1 71.0 mm to (126.0, 31.3), turned to -90 degrees
- moved Nes1 43.7 mm to (169.2, 106.3), turned to -90 degrees
- moved A1 40.5 mm to (142.7, 67.3), turned to -90 degrees
- moved Snes1 23.0 mm to (151.6, 70.3), turned to 90 degrees
Connections:
- A1 pad 29: unconnected-(A1-GND-Pad29) -> Net-(3v3_regulator1-GND)
- A1 pad 4: Net-(Nes1-GND) -> Net-(3v3_regulator1-GND)
- C1 pad 2: Net-(U1-GND) -> Net-(3v3_regulator1-GND)
- Nes1 pad 2: Net-(A1-D4) -> Net-(A1-D6)
- Nes1 pad 4: Net-(A1-D6) -> Net-(A1-D4)
- Nes1 pad 7: Net-(Nes1-GND) -> Net-(3v3_regulator1-GND)
- Snes1 pad 2: Net-(A1-D4) -> Net-(A1-D6)
- Snes1 pad 4: Net-(A1-D6) -> Net-(A1-D4)
- Snes1 pad 7: Net-(Nes1-GND) -> Net-(3v3_regulator1-GND)
Routing:
- net Net-(3v3_regulator1-GND): track 0.00 -> 232.2 mm
- net Net-(3v3_regulator1-VI): track 0.00 -> 187.1 mm
- net Net-(A1-D2): track 0.00 -> 85.5 mm
- net Net-(A1-D3): track 0.00 -> 84.9 mm
- net Net-(A1-D6): track 0.00 -> 83.8 mm
- net Net-(A1-D5): track 0.00 -> 78.2 mm
- net Net-(A1-D13): track 0.00 -> 76.3 mm
- net Net-(A1-D4): track 0.00 -> 74.0 mm
- net Net-(A1-D9): track 0.00 -> 43.8 mm
- net Net-(A1-D11): track 0.00 -> 43.4 mm
- net Net-(A1-D12): track 0.00 -> 41.2 mm
- net Net-(A1-D8): track 0.00 -> 37.6 mm
- net Net-(A1-D7): track 0.00 -> 32.5 mm
- net Net-(A1-A5): track 0.00 -> 29.8 mm
- net Net-(A1-A4): track 0.00 -> 25.2 mm
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