File: projects/5v radio/5v radio.kicad_pcb (KiCad board)
At the start: 2 copper layers, 8 parts

Commit message: update
Other:
- board text added: "CRJ"
Changed lines of the file:
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@@
 		(fp_arc
 			(start 5.850318 14.881681)
-			(mid 4.53186 15.762642)
+			(mid 4.531861 15.762643)
 			(end 2.976637 16.072)
 			(stroke
@@
 		(layer "F.SilkS")
 	)
+	(gr_text "CRJ"
+		(at 113.03 81.026 0)
+		(layer "F.SilkS")
+		(effects
+			(font
+				(size 10 10)
+				(thickness 0.3)
+				(bold yes)
+			)
+			(justify left bottom)
+		)
+	)
 	(segment
