File: projects/remote controll/remote controll.kicad_pcb (KiCad board)
At the start: 2 copper layers, 13 parts, among them U1 L7805

Commit message: update
Parts:
- removed C1, C2, C3: C_Polarized, Capacitor_THT:CP_Radial_D8.0mm_P3.80mm
- added C12v1: C_Polarized, Capacitor_THT:CP_Radial_D8.0mm_P3.80mm, F.Cu at (93.0, 52.3)
- added C3.3v1: C_Polarized, Capacitor_THT:CP_Radial_D8.0mm_P3.80mm, F.Cu at (100.6, 79.8)
- added C5v1: C_Polarized, Capacitor_THT:CP_Radial_D8.0mm_P3.80mm, F.Cu at (100.6, 64.0)
- added D1: LED, LED_THT:LED_D5.0mm, F.Cu at (194.4, 65.0)
- added D2: LED, LED_THT:LED_D5.0mm, F.Cu at (194.4, 72.5)
- added D3: LED, LED_THT:LED_D5.0mm, F.Cu at (194.6, 80.0)
- added D4: LED, LED_THT:LED_D5.0mm, F.Cu at (194.6, 87.1)
- added R1: R, Resistor_THT:R_Axial_DIN0204_L3.6mm_D1.6mm_P7.62mm_Horizontal, F.Cu at (194.2, 49.5)
- added R2: R, Resistor_THT:R_Axial_DIN0204_L3.6mm_D1.6mm_P7.62mm_Horizontal, F.Cu at (191.0, 49.5)
- added R3: R, Resistor_THT:R_Axial_DIN0204_L3.6mm_D1.6mm_P7.62mm_Horizontal, F.Cu at (187.9, 49.5)
- added R4: R, Resistor_THT:R_Axial_DIN0204_L3.6mm_D1.6mm_P7.62mm_Horizontal, F.Cu at (184.7, 49.5)
- moved MOTOR_B1 95.8 mm to (66.8, 28.7)
- moved MOTOR_A1 95.3 mm to (66.8, 41.9)
- moved POWER_INPUT1 90.8 mm to (83.7, 54.9)
- moved GPS1 89.1 mm to (156.9, 25.8)
- moved TB6612FNG1 88.8 mm to (122.2, 27.1)
- moved NRF1 53.0 mm to (103.0, 96.8), turned to 180 degrees
- moved 3v3_regulator1 42.1 mm to (90.8, 80.8)
- moved U1 31.3 mm to (90.8, 68.8)
- moved MPU1 31.2 mm to (172.1, 49.6)
- moved A1 22.9 mm to (126.7, 58.4)
Connections:
- A1 pad 21: unconnected-(A1-A2-Pad21) -> Net-(A1-A2)
- A1 pad 22: unconnected-(A1-A3-Pad22) -> Net-(A1-A3)
- A1 pad 25: unconnected-(A1-A6-Pad25) -> Net-(A1-A6)
- A1 pad 26: unconnected-(A1-A7-Pad26) -> Net-(A1-A7)
- A1 pad 27: unconnected-(A1-+5V-Pad27) -> Net-(A1-+5V)
- A1 pad 29: unconnected-(A1-GND-Pad29) -> Net-(3v3_regulator1-GND)
- A1 pad 30: Net-(A1-VIN) -> unconnected-(A1-VIN-Pad30)
- A1 pad 4: unconnected-(A1-GND-Pad4) -> Net-(3v3_regulator1-GND)
- GPS1 pad 4: Net-(A1-VIN) -> Net-(A1-+5V)
- MPU1 pad 1: Net-(A1-VIN) -> Net-(A1-+5V)
- TB6612FNG1 pad 2: Net-(A1-VIN) -> Net-(A1-+5V)
- U1 pad 3: Net-(A1-VIN) -> Net-(A1-+5V)
