File: projects/remote controll/remote controll.kicad_sch (KiCad schematic)
At the start: 13 parts, among them U1 L7805

Commit message: update
Parts:
- added D1, D2, D3, D4: LED, LED_THT:LED_D5.0mm, symbol Device:LED
- added R1, R2, R3, R4: R, Resistor_THT:R_Axial_DIN0204_L3.6mm_D1.6mm_P7.62mm_Horizontal, symbol Device:R
- renumbered C1 to C12v1, C3 to C3.3v1, C2 to C5v1
Connections:
- net at 3v3_regulator1.1 (GND), C12v1.2, C3.3v1.2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: now also A1.29 (GND), A1.4 (GND), R1.2, R2.2, R3.2, R4.2
- net at A1.21 (A2): now also D4.1 (K)
- net at A1.22 (A3): now also D1.1 (K)
- net at A1.25 (A6): now also D2.1 (K)
- net at A1.26 (A7): now also D3.1 (K)
- net at A1.27 (+5V): now also C5v1.1, GPS1.4 (VCC), MPU1.1 (VCC), TB6612FNG1.2 (VCC), U1.3 (OUT)
- new net: D1.2 (A), R1.1
- new net: D4.2 (A), R4.1
- new net: D2.2 (A), R2.1
- new net: D3.2 (A), R3.1
- now unconnected: A1.30 (VIN)
Other:
- moved on the sheet: 3v3_regulator1, A1, C12v1, C3.3v1, C5v1, GPS1, MOTOR_A1, MOTOR_B1, MPU1, NRF1, POWER_INPUT1, TB6612FNG1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
