File: projects/remote controll/remote controll_v4.kicad_pcb (KiCad board)
At the start: 2 copper layers, 23 parts, among them U1 L7805

Commit message: 5V DONE
Parts:
- removed REF** (x4): MountingHole_3.2mm_M3_ISO7380, MountingHole:MountingHole_3.2mm_M3_ISO7380
- moved C3.3v1 66.3 mm to (206.6, 89.9), turned to -90 degrees
- moved C12v1 65.8 mm to (145.3, 115.1), turned to 0 degrees
- moved D1 16.0 mm to (216.7, 89.7), turned to -90 degrees
- moved R3 14.7 mm to (221.5, 104.6)
- moved R1 13.9 mm to (228.9, 91.2), turned to 180 degrees
- moved D3 10.2 mm to (216.7, 102.6), turned to -90 degrees
- moved C5v1 4.26 mm to (197.0, 89.9)
- moved D2 3.15 mm to (216.7, 96.0), turned to -90 degrees
- moved MOTOR_A1 2.35 mm to (194.8, 62.5)
- moved 3v3_regulator1 1.45 mm to (149.6, 122.3)
- moved R2 1.37 mm to (221.2, 97.8)
- moved TB6612FNG1 1.21 mm to (171.6, 93.0)
- moved U1 0.95 mm to (191.4, 78.7)
- moved GPS1 0.85 mm to (212.2, 124.7)
- moved A1 0.70 mm to (176.0, 100.7)
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Connections:
- A1 pad 21: unconnected-(A1-A2-Pad21) -> Net-(A1-A2)
Routing:
- net Net-(A1-+5V): track 147.0 -> 0.00 mm
- net Net-(3v3_regulator1-GND): track 328.0 -> 186.8 mm
- net Net-(A1-D2): track 99.5 -> 0.00 mm
- net Net-(A1-D10): track 97.9 -> 0.00 mm
- net Net-(A1-D3): track 81.9 -> 0.00 mm
- net Net-(A1-A1): track 77.9 -> 0.00 mm
- net Net-(A1-D13): track 76.2 -> 0.00 mm
- net Net-(A1-A0): track 67.4 -> 0.00 mm
- net Net-(A1-D7): track 63.1 -> 0.00 mm
- net Net-(A1-A4): track 57.7 -> 0.00 mm
- net Net-(A1-D6): track 57.5 -> 0.00 mm
- net Net-(A1-A5): track 54.1 -> 0.00 mm
- net Net-(A1-D11): track 52.5 -> 0.00 mm
- net Net-(A1-D9): track 50.9 -> 0.00 mm
- net Net-(A1-D5): track 49.4 -> 0.00 mm
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Other:
- board text removed: "+"
- board text removed: "-"
