File: projects/remote controll/remote controll_v1.kicad_pcb (KiCad board)
At the start: 2 copper layers, 23 parts, among them U1 L7805

Commit message: a lot of project updates
Other:
- board text added: "CRJ"

Commit message: and to the factory it goes
Routing:
- net Net-(3v3_regulator1-GND): track 328.0 -> 343.4 mm
- net Net-(A1-D13): track 76.2 -> 81.7 mm
- net Net-(3v3_regulator1-VI): track 184.9 -> 182.0 mm
- net Net-(A1-+5V): track 147.0 -> 149.3 mm
