File: projects/pro micro nintendo adapter/pro micro nintendo adapter.kicad_pcb (KiCad board)
At the start: 2 copper layers, 25 x 105 mm, 6 parts

Commit message: and to the factory it goes
Parts:
- added REF**: MountingHole_2.2mm_M2, MountingHole:MountingHole_2.2mm_M2, F.Cu at (121.9, 112.8)
- added REF**: MountingHole_2.2mm_M2, MountingHole:MountingHole_2.2mm_M2, F.Cu at (140.5, 81.0)
- added REF**: MountingHole_2.2mm_M2, MountingHole:MountingHole_2.2mm_M2, F.Cu at (131.6, 48.3)
- added REF**: MountingHole_2.2mm_M2, MountingHole:MountingHole_2.2mm_M2, F.Cu at (141.2, 112.8)
- added REF**: MountingHole_2.2mm_M2, MountingHole:MountingHole_2.2mm_M2, F.Cu at (121.7, 143.5)
- added REF**: MountingHole_2.2mm_M2, MountingHole:MountingHole_2.2mm_M2, F.Cu at (141.5, 143.5)
- added REF**: MountingHole_2.2mm_M2, MountingHole:MountingHole_2.2mm_M2, F.Cu at (122.7, 81.0)
Routing:
- net Net-(U1-SDA): track 95.8 -> 86.1 mm
- net Net-(U1-SCL): track 83.5 -> 81.8 mm
- net Net-(U1-7): track 58.4 -> 59.3 mm
