File: projects/nano breakout/nano breakout/nano breakout.kicad_pcb (KiCad board)
At the start: 2 copper layers, 1 part

Commit message: footprint library
Routing:
- net (no net): track 0.00 -> 510.5 mm
